Commit message: updated Lab 6

File: laboratory/Lab6/urdf/fingeredu.urdf (robot description, URDF)
Before this commit: robot fingeredu, 6 links, 5 joints
Links:
- link base_link: mass 0.2 -> 1
- link finger_base_link: mass 0.2 -> 1
Joints:
- joint finger_upper_to_middle_joint: limit lower=-3.14 upper=3.14 effort=1000 velocity=1000 -> lower=-3.14159265359 upper=3.14159265359 effort=1000 velocity=1000
