Commit message: updated lab5

File: laboratory/Lab5/urdf/fingeredu.urdf (robot description, URDF)
Before this commit: robot fingeredu, 6 links, 5 joints
Joints:
- joint finger_upper_to_middle_joint: limit lower=-1.57079632679 upper=1.57079632679 effort=1000 velocity=1000 -> lower=-3.14159265359 upper=3.14159265359 effort=1000 velocity=1000

Commit message: Lab 5

File: laboratory/Lab5/urdf/fingeredu.urdf (robot description, URDF)
Before this commit: robot fingeredu, 6 links, 5 joints
Links:
- link base_link: mass 1 -> 0.2
- link finger_base_link: mass 1 -> 0.2; geometry visual mesh filename=package://meshes/base_back.stl scale=1 1 1; visual mesh filename=package://meshes/base_front.stl scale=1 1 1
Joints:
- joint finger_upper_to_middle_joint: limit lower=-3.14159265359 upper=3.14159265359 effort=1000 velocity=1000 -> lower=-3.14 upper=3.14 effort=1000 velocity=1000
